Commit message: pid controller for unbalened chassis

File: src/ouster_OS1_LiDar/ouster_description/urdf/OS1-64.urdf.xacro (robot description, xacro)
@@ -2,5 +2,5 @@
 <robot xmlns:xacro="http://www.ros.org/wiki/xacro" name="OS1-64">
   <xacro:property name="M_PI" value="3.1415926535897931" />
-  <xacro:macro name="OS1-64" params="*origin parent:=Rover_frame name:=os1_sensor topic_points:=/os1_cloud_node/points topic_imu:=/os1_cloud_node/imu hz:=10 lasers:=64 samples:=512 min_range:=0.9 max_range:=75.0 noise:=0.008 min_angle:=-${M_PI} max_angle:=${M_PI} lidar_link:=os1_lidar imu_link:=os1_imu vfov_min:=-.26 vfov_max:=.26">
+  <xacro:macro name="OS1-64" params="*origin parent:=CHASSIS name:=os1_sensor topic_points:=/os1_cloud_node/points topic_imu:=/os1_cloud_node/imu hz:=10 lasers:=64 samples:=512 min_range:=0.9 max_range:=75.0 noise:=0.008 min_angle:=-${M_PI} max_angle:=${M_PI} lidar_link:=os1_lidar imu_link:=os1_imu vfov_min:=-.26 vfov_max:=.26">
     <joint name="${name}_mount_joint" type="fixed">
       <xacro:insert_block name="origin" />

File: src/rover_description/urdf/Rover_URDF_V6.urdf.xacro (robot description, xacro)
@@ -6,9 +6,24 @@
      -->
 <robot xmlns:xacro="http://www.ros.org/wiki/xacro" name="rover">
-  <link
-    name="Rover_frame">
-    <inertial>
-      <origin
-        xyz="-0.18 0.00 -0.105"
+  <!-- virtual joint - link pair to get the inclination of the rover base -->
+  <joint name="Base_joint" type="revolute">
+      <origin
+      xyz="-0.18 0 -0.105"
+      rpy="0 0 0" />
+      <axis
+      xyz="0 1 0" />
+      <limit
+      lower="-1.57"
+      upper="1.57"
+      effort="100"
+      velocity="10" />
+      <parent link="CHASSIS"/>
+      <child link="ROVER_FRAME"/>
+  </joint>
+  <link
+    name="ROVER_FRAME">
+    <inertial>
+      <origin
+        xyz="0 0 0"
         rpy="0 0 0" />
       <mass
@@ -22,25 +37,43 @@
         izz="0.290474747721043" />
     </inertial>
-    <visual>
-      <origin
-        xyz="0 0 0"
-        rpy="0 0 0" />
-      <geometry>
-        <mesh
-          filename="package://rover_description/meshes/Rover frame.STL" />
-      </geometry>
-      <material
-        name="">
-        <color
-          rgba="0.792156862745098 0.819607843137255 0.933333333333333 1" />
-      </material>
-    </visual>
-    <collision>
-      <origin
-        xyz="0 0 0"
-        rpy="0 0 0" />
-      <geometry>
-        <mesh
-          filename="package://rover_description/meshes/Rover frame.STL" />
+  </link>
+<!--                                                                     -->
+  <link
+    name="CHASSIS">
+    <inertial>
+      <origin
+        xyz="-0.18 0.00 -0.105"
+        rpy="0 0 0" />
+      <mass
+        value="2.86544274049469" />
+      <inertia
+        ixx="0.103079825863941"
+        ixy="-0.00028741576657649"
+        ixz="-0.024219701014768"
+        iyy="0.230618546322903"
+        iyz="-8.00119839628446E-05"
+        izz="0.290474747721043" />
+    </inertial>
+    <visual>
+      <origin
+        xyz="0 0 0"
+        rpy="0 0 0" />
+      <geometry>
+        <mesh
+          filename="package://rover_description/meshes/CHASSIS.STL" />
+      </geometry>
+      <material
+        name="">
+        <color
+          rgba="0.792156862745098 0.819607843137255 0.933333333333333 1" />
+      </material>
+    </visual>
+    <collision>
+      <origin
+        xyz="0 0 0"
+        rpy="0 0 0" />
+      <geometry>
+        <mesh
+          filename="package://rover_description/meshes/CHASSIS.STL" />
       </geometry>
     </collision>
@@ -90,8 +123,8 @@
     type="revolute">
     <origin
-      xyz="-0.18 0.23 -0.105"
-      rpy="0 0 0" />
-    <parent
-      link="Rover_frame" />
+      xyz="0 0.23 0"
+      rpy="0 0 0" />
+    <parent
+      link="ROVER_FRAME" />
     <child
       link="ROCKER_LEFT" />
@@ -99,6 +132,6 @@
       xyz="0 -1 0" />
     <limit
-      lower="-0.01"
-      upper="0.01"
+      lower="-3.14"
+      upper="3.14"
       effort="100"
       velocity="30" />
@@ -366,8 +399,8 @@
     type="revolute">
     <origin
-      xyz="-0.18 -0.23 -0.105"
-      rpy="0 0 0" />
-    <parent
-      link="Rover_frame" />
+      xyz="0 -0.23 0"
+      rpy="0 0 0" />
+    <parent
+      link="ROVER_FRAME" />
     <child
       link="ROCKER_RIGHT" />
@@ -601,5 +634,5 @@
     <axis xyz="0 1 0" />
     <origin xyz=".15 0 .1" rpy="0 0 0"/>
-    <parent link="Rover_frame"/>
+    <parent link="CHASSIS"/>
     <child link="hokuyo"/>
   </joint>
@@ -623,5 +656,5 @@
   <!-- LiDar -->
   <xacro:include filename="$(find ouster_description)/urdf/OS1-64.urdf.xacro"/>
-  <OS1-64 parent="Rover_frame" name="os1_sensor" hz="10" samples="220" lasers="64" min_range="0.1" max_range="10.0">
+  <OS1-64 parent="CHASSIS" name="os1_sensor" hz="10" samples="220" lasers="64" min_range="0.1" max_range="10.0">
     <origin xyz="0 0 0.5" rpy="0 0 0" />
   </OS1-64>
@@ -706,5 +739,5 @@
      <odometryTopic>odom</odometryTopic>
      <odometryFrame>odom</odometryFrame>
-     <robotBaseFrame>Rover_frame</robotBaseFrame>
+     <robotBaseFrame>CHASSIS</robotBaseFrame>
      <odometrySource>world</odometrySource>
      <publishTf>1</publishTf>
@@ -713,5 +746,5 @@
     <alwaysOn>true</alwaysOn>
     <updateRate>50.0</updateRate>
-    <bodyName>Rover_frame</bodyName>
+    <bodyName>CHASSIS</bodyName>
     <topicName>odom</topicName>
     <gaussianNoise>0.01</gaussianNoise>
@@ -722,5 +755,5 @@
   <plugin name="joint_state_publisher" filename="libgazebo_ros_joint_state_publisher.so">
     <robotNamespace>/rover</robotNamespace>
-    <jointName>BOGIE_LEFT , BOGIE_RIGHT , ROCKER_RIGHT </jointName>
+    <jointName>Base_joint, BOGIE_LEFT , BOGIE_RIGHT , ROCKER_RIGHT </jointName>
     <updateRate>100.0</updateRate>
     <alwaysOn>true</alwaysOn>
