Commit message: added damping factor to two joints (bogie left and right)

File: src/rover_description/urdf/Rover_URDF_V6.urdf.xacro (robot description, xacro)
@@ -214,4 +214,5 @@
       effort="0"
       velocity="0" />
+    <dynamics damping ="50"/>
   </joint>
   <link
@@ -489,4 +490,5 @@
       effort="0"
       velocity="0" />
+    <dynamics damping ="50"/>
   </joint>
   <link

Commit message: path planner

File: src/rover_description/urdf/Rover_URDF_V6.urdf.xacro (robot description, xacro)
@@ -598,4 +598,27 @@
       xyz="0 -1 0" />
   </joint>
+  <joint name="hokuyo_joint" type="fixed">
+    <axis xyz="0 1 0" />
+    <origin xyz=".15 0 .1" rpy="0 0 0"/>
+    <parent link="Rover_frame"/>
+    <child link="hokuyo"/>
+  </joint>
+  <!-- Hokuyo Laser -->
+  <link name="hokuyo">
+    <collision>
+      <origin xyz="0 0 0" rpy="0 0 0"/>
+      <geometry>
+    <box size="0.1 0.1 0.1"/>
+      </geometry>
+    </collision>
+    <visual>
+      <origin xyz="0 0 0" rpy="0 0 0"/>
+    </visual>
+    <inertial>
+      <mass value="1e-5" />
+      <origin xyz="0 0 0" rpy="0 0 0"/>
+      <inertia ixx="1e-6" ixy="0" ixz="0" iyy="1e-6" iyz="0" izz="1e-6" />
+    </inertial>
+  </link>
   <!-- LiDar -->
   <xacro:include filename="$(find ouster_description)/urdf/OS1-64.urdf.xacro"/>

Commit message: artag and camera added

File: src/rover_description/urdf/Rover_URDF_V6.urdf.xacro (robot description, xacro)
@@ -659,4 +659,72 @@
     <origin xyz="0 0 0.5" rpy="0 0 0" />
   </OS1-64>
+<!-- camera -->
+  <gazebo reference="camera_link">
+    <sensor type="camera" name="camera1">
+      <update_rate>30.0</update_rate>
+      <camera name="head">
+        <horizontal_fov>1.3962634</horizontal_fov>
+        <image>
+          <width>800</width>
+          <height>800</height>
+          <format>R8G8B8</format>
+        </image>
+        <clip>
+          <near>0.02</near>
+          <far>300</far>
+        </clip>
+        <noise>
+          <type>gaussian</type>
+          <!-- Noise is sampled independently per pixel on each frame.
+               That pixel's noise value is added to each of its color
+               channels, which at that point lie in the range [0,1]. -->
+          <mean>0.0</mean>
+          <stddev>0.007</stddev>
+        </noise>
+      </camera>
+      <plugin name="camera_controller" filename="libgazebo_ros_camera.so">
+        <alwaysOn>true</alwaysOn>
+        <updateRate>0.0</updateRate>
+        <cameraName>camera1</cameraName>
+        <imageTopicName>image_raw</imageTopicName>
+        <cameraInfoTopicName>camera_info</cameraInfoTopicName>
+        <frameName>camera_link</frameName>
+        <hackBaseline>0.07</hackBaseline>
+        <distortionK1>0.0</distortionK1>
+        <distortionK2>0.0</distortionK2>
+        <distortionK3>0.0</distortionK3>
+        <distortionT1>0.0</distortionT1>
+        <distortionT2>0.0</distortionT2>
+      </plugin>
+    </sensor>
+  </gazebo>
+<!-- Camera -->
+ <link name="camera_link">
+    <inertial>
+      <origin xyz="0 0 0" rpy="0 0 0" />
+      <mass value="1" />
+      <!-- RANDOM INERTIA BELOW -->
+      <inertia ixx="1e-6" ixy="0" ixz="0" iyy="1e-6" iyz="0" izz="1e-6" />
+    </inertial>
+    <visual>
+      <origin xyz="0 0 0" rpy="0 0 0" />
+      <geometry>
+        <box size="0.05 0.07 0.05"/>
+      </geometry>
+      <material name="white" />
+    </visual>
+    <collision>
+      <origin xyz="0 0 0" rpy="0 0 0"/>
+      <geometry>
+        <box size="0.05 0.07 0.05"/>
+      </geometry>
+    </collision>
+  </link>
+  <joint name="camera_joint" type="fixed">
+  <axis xyz="0 1 0" />
+    <origin xyz="0 0 0.2" rpy="0 0 0"/>
+    <parent link="CHASSIS"/>
+    <child link="camera_link"/>
+  </joint>
 <!-- For ros_control -->
 <transmission name="transmission_rocker_left">  <!-- with left rocker -->

Commit message: AR tag added to the wolrd

File: src/rover_description/urdf/Rover_URDF_V6.urdf.xacro (robot description, xacro)
@@ -14,6 +14,6 @@
       xyz="0 1 0" />
       <limit
-      lower="-1.57"
-      upper="1.57"
+      lower="-0.1"
+      upper="0.1"
       effort="100"
       velocity="10" />
@@ -136,4 +136,5 @@
       effort="100"
       velocity="30" />
+      <dynamics friction="10000"/>
   </joint>
   <link
@@ -247,5 +248,5 @@
       effort="0"
       velocity="0" />
-    <dynamics damping ="50"/>
+    <dynamics friction="10"/>
   </joint>
   <link
@@ -412,4 +413,5 @@
       effort="0"
       velocity="0" />
+      <dynamics friction="10000"/>
   </joint>
   <link
@@ -523,5 +525,5 @@
       effort="0"
       velocity="0" />
-    <dynamics damping ="50"/>
+    <dynamics friction="10"/>
   </joint>
   <link
@@ -703,5 +705,5 @@
     <inertial>
       <origin xyz="0 0 0" rpy="0 0 0" />
-      <mass value="1" />
+      <mass value="1e-5" />
       <!-- RANDOM INERTIA BELOW -->
       <inertia ixx="1e-6" ixy="0" ixz="0" iyy="1e-6" iyz="0" izz="1e-6" />
